Commit message: mise a jour + map

File: description/camera.xacro (robot description, xacro)
@@ -30,5 +30,5 @@
             <pose>0 0 0 0 0 0</pose>
             <update_rate>30</update_rate>
-            <visualize>true</visualize>
+            <visualize>false</visualize>
             <camera>
                 <horizontal_fov>1.047</horizontal_fov>

File: description/control.xacro (robot description, xacro)
@@ -9,6 +9,6 @@
             <wheel_diameter>0.1</wheel_diameter>
             <!--limits of the wheels (torq)-->
-            <max_wheel_torque>200</max_wheel_torque>
-            <max_wheel_acceleration>10.0</max_wheel_acceleration>
+            <max_wheel_torque>250</max_wheel_torque>
+            <max_wheel_acceleration>50.0</max_wheel_acceleration>
             <!--output-->
             <odometry_frame>odom</odometry_frame>

File: description/lidar.xacro (robot description, xacro)
@@ -27,5 +27,5 @@
         <sensor name = 'laser' type = 'ray'>
             <pose> 0 0 0 0 0 0 </pose>
-            <visualize>false</visualize>
+            <visualize>true</visualize>
             <update_rate>10</update_rate>
             <ray>

File: description/robot_include.xacro (robot description, xacro)
@@ -21,4 +21,10 @@
     <link name = "base_link">
     </link>
+    <joint name = "base_footprint_joint" type = "fixed">
+        <parent link ="base_link"/>
+        <child link ="base_footprint"/>
+        <origin xyz = "0 0 0" rpy = "0 0 0"/>
+    </joint>
+    <link name = "base_footprint" />
     <joint name = "base_to_chassis" type = "fixed">
         <origin xyz = "-0.1 0 0" rpy = "0 0 0"/>
